File: GBAKicad/GBAKicad.kicad_sch (KiCad schematic)
At the start: 63 parts, among them J1 USB_C_Receptacle_USB2.0_16P, J2 BATT_Conn, J3 Jumper, J4 OLED_Conn, Q2 PMOS, SW1 EN, SW10 SW_Push, SW11 SW_Push, SW12 SW_Push, SW13 SW_Push, SW14 SW_Push, SW15 SW_Push, SW16 BTN_SYS, SW2 SW_SPDT, SW3 BOOT, SW4 SW_Push, SW5 SW_Push, SW6 SW_Push, SW7 SW_Push, SW8 SW_Push, SW9 SW_Push, U1 ESP32-S3-WROOM-1, U2 MIC5219-3.3YM5, U3 TP4056-42-ESOP8, U4 DW01A, U5 AMS1117-3.3

Commit message: updating the PCB
Parts:
- J2: footprint (none) -> Connector_JST:JST_ZH_S2B-ZR-SM4A-TF_1x02-1MP_P1.50mm_Horizontal
- J3, R1, R10, R11, R12, R13, R14, R15, R16, R17, R2, R3, R4, R5, R6, R7, R8, R9: footprint (none) -> Resistor_SMD:R_0603_1608Metric
- J4: footprint (none) -> custom_footprints:OLED128x32_1x04_P2.54mm_socket
- Q1: footprint Custom Footprints:SOT-23-6L_TCP -> custom_footprints:SOT-23-6L_TCP
- Q2: footprint (none) -> Package_TO_SOT_SMD:SOT-23
- SW1: footprint (none) -> Button_Switch_SMD:SW_SPST_TS-1088-xR020
- SW10: value SW_Push -> BTN_R; footprint (none) -> custom_footprints:TS-1224VW
- SW11: value SW_Push -> BTN_X; footprint (none) -> custom_footprints:SW_PUSH_8mm_H5mm_custom
- SW12: value SW_Push -> BTN_A; footprint (none) -> custom_footprints:SW_PUSH_8mm_H5mm_custom
- SW13: value SW_Push -> BTN_B; footprint (none) -> custom_footprints:SW_PUSH_8mm_H5mm_custom
- SW14: value SW_Push -> BTN_Y; footprint (none) -> custom_footprints:SW_PUSH_8mm_H5mm_custom
- SW15: value SW_Push -> BTN_SELECT; footprint (none) -> custom_footprints:SW_PUSH_8mm_H5mm_custom
- SW16: footprint (none) -> custom_footprints:SW_PUSH_8mm_H5mm_custom
- SW2: value SW_SPDT -> SW_PWR; footprint (none) -> Connector_PinSocket_2.54mm:PinSocket_1x03_P2.54mm_Vertical
- SW3: footprint (none) -> custom_footprints:SW_SPST_TS-1088-xR020
- SW4: value SW_Push -> BTN_L; footprint (none) -> custom_footprints:TS-1224VW
- SW5: value SW_Push -> BTN_UP; footprint (none) -> custom_footprints:SW_PUSH_8mm_H5mm_custom
- SW6: value SW_Push -> BTN_LEFT; footprint (none) -> custom_footprints:SW_PUSH_8mm_H5mm_custom
- SW7: value SW_Push -> BTN_DOWN; footprint (none) -> custom_footprints:SW_PUSH_8mm_H5mm_custom
- SW8: value SW_Push -> BTN_RIGHT; footprint (none) -> custom_footprints:SW_PUSH_8mm_H5mm_custom
- SW9: value SW_Push -> BTN_START; footprint (none) -> custom_footprints:SW_PUSH_8mm_H5mm_custom
- TP1, TP3, TP4, TP5: footprint (none) -> TestPoint:TestPoint_Pad_D2.0mm
Connections:
- net BAT_CHECK is gone; now on net BATT_CHECK: U1.4 (IO4)
- net +5V: now also C8.1
- net +BATT: now also C10.2; no longer C10.1
- net BTN_X: no longer SW14.2
- net BTN_Y: now also SW14.2
- net GND: now also C10.1; no longer C10.2
- net at D2.1 (K), U3.6 (~{STDBY}): no longer C8.1
Other:
- moved on the sheet: C10, C8

Commit message: pcb change
Connections:
- net BTN_Sys is gone; now on net BTN_SYS: U1.33 (IO40)
Changed lines of the file:
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@@
 		)
 	)
-	(global_label "BTN_Sys"
+	(global_label "BTN_SYS"
 		(shape input)
 		(at 55.88 67.31 0)
@@
 		)
 		(property "Intersheetrefs" "${INTERSHEET_REFS}"
-			(at 66.6061 67.31 0)
+			(at 66.9085 67.31 0)
 			(hide yes)
 			(show_name no)
